File: PCB/Cbot2.kicad_pcb (KiCad board)
At the start: 4 copper layers, 65 x 56 mm, 26 parts, among them J1 +5V Power, J10 Pads, J11 Pads, J12 Pads, J2 +5V RPi Power, J3 Raspberry_Pi_2_3, J4 Lights, J5 Fan, J6 Switch, J7 Amplifier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

Commit message: PCB update
Move signal from Raspberry Pi pin 12 to pin 11.
Connections:
- J3 pad 11: Net-(J3-Pad11) -> FAN
- J3 pad 12: PWM0 -> Net-(J3-Pad12)
- R1 pad 2: PWM0 -> FAN
Routing:
- net PWM0: track 11.4 -> 0.00 mm
- net FAN: track 0.00 -> 8.83 mm
Other:
- board text added: "CordeBot 2.0 01/26/2020"
- board text removed: "CordeBot 2.0 12/2019"
